File: LAN8742A-breakout.kicad_pcb (KiCad board)
At the start: 6 copper layers, 0 parts

Commit message: routed signals
Parts:
- added C1: 4.7µF, Capacitor_SMD:C_0603_1608Metric_Pad1.08x0.95mm_HandSolder, F.Cu at (143.8, 75.7)
- added C10: 33pF, Capacitor_SMD:C_0603_1608Metric_Pad1.08x0.95mm_HandSolder, F.Cu at (136.9, 78.5)
- added C11: 33pF, Capacitor_SMD:C_0603_1608Metric_Pad1.08x0.95mm_HandSolder, F.Cu at (140.1, 75.3)
- added C2: 100nF, Capacitor_SMD:C_0603_1608Metric_Pad1.08x0.95mm_HandSolder, F.Cu at (144.9, 74.6)
- added C3: 100nF, Capacitor_SMD:C_0603_1608Metric_Pad1.08x0.95mm_HandSolder, F.Cu at (152.1, 80.0)
- added C4: 4.7µF, Capacitor_SMD:C_0603_1608Metric_Pad1.08x0.95mm_HandSolder, F.Cu at (153.2, 78.9)
- added C5: 100nF, Capacitor_SMD:C_0603_1608Metric_Pad1.08x0.95mm_HandSolder, F.Cu at (139.0, 81.3)
- added C6: 4.7µF, Capacitor_SMD:C_0603_1608Metric_Pad1.08x0.95mm_HandSolder, F.Cu at (137.8, 82.4)
- added C7: 1µF, Capacitor_SMD:C_0603_1608Metric_Pad1.08x0.95mm_HandSolder, F.Cu at (140.3, 78.9)
- added C8: 470pF, Capacitor_SMD:C_0603_1608Metric_Pad1.08x0.95mm_HandSolder, F.Cu at (141.4, 80.1)
- added C9: 4.7µF, Capacitor_SMD:C_0603_1608Metric_Pad1.08x0.95mm_HandSolder, F.Cu at (130.5, 57.4)
- added FB1: FerriteBead, 0_oscillators:L0603, F.Cu at (162.9, 86.5)
- added H1: MountingHole, MountingHole:MountingHole_3.2mm_M3_DIN965, F.Cu at (130.3, 49.0)
- added H2: MountingHole, MountingHole:MountingHole_3.2mm_M3_DIN965, F.Cu at (164.3, 49.0)
- added H3: MountingHole, MountingHole:MountingHole_3.2mm_M3_DIN965, F.Cu at (164.3, 93.0)
- added H4: MountingHole, MountingHole:MountingHole_3.2mm_M3_DIN965, F.Cu at (130.3, 93.0)
- added J1: HR911105A_C12074, 0_connector:RJ45-TH_HR911105A, F.Cu at (147.3, 54.7)
- added J2: J_RMII, Connector_PinHeader_2.54mm:PinHeader_2x10_P2.54mm_Vertical, F.Cu at (158.7, 91.4)
- added J3: J_POW, Connector_PinHeader_2.54mm:PinHeader_1x03_P2.54mm_Vertical, F.Cu at (165.7, 87.1)
- added J4: J_LED, Connector_PinSocket_2.54mm:PinSocket_1x02_P2.54mm_Vertical, F.Cu at (165.7, 75.0)
- added JP1: REGOFF, Jumper:SolderJumper-2_P1.3mm_Open_RoundedPad1.0x1.5mm, F.Cu at (165.7, 62.0)
- added JP2: nINTSEL, Jumper:SolderJumper-2_P1.3mm_Bridged_RoundedPad1.0x1.5mm, F.Cu at (165.7, 70.2)
- added JP3: nINTSEL, Jumper:SolderJumper-2_P1.3mm_Open_RoundedPad1.0x1.5mm, F.Cu at (165.7, 67.7)
- added JP4: SH, Jumper:SolderJumper-2_P1.3mm_Bridged_RoundedPad1.0x1.5mm, F.Cu at (136.3, 55.8)
- added JP5: SH, Jumper:SolderJumper-2_P1.3mm_Bridged_RoundedPad1.0x1.5mm, F.Cu at (158.3, 55.7)
- added R1: 12.1k, Resistor_SMD:R_0603_1608Metric_Pad0.98x0.95mm_HandSolder, F.Cu at (143.9, 71.3)
- added R10: 49.9, Resistor_SMD:R_0603_1608Metric_Pad0.98x0.95mm_HandSolder, F.Cu at (144.4, 68.0)
- added R11: 49.9, Resistor_SMD:R_0603_1608Metric_Pad0.98x0.95mm_HandSolder, F.Cu at (152.7, 69.6)
- added R12: 49.9, Resistor_SMD:R_0603_1608Metric_Pad0.98x0.95mm_HandSolder, F.Cu at (149.6, 68.1)
- added R2: 10k, Resistor_SMD:R_0603_1608Metric_Pad0.98x0.95mm_HandSolder, F.Cu at (165.7, 72.3)
- added R3: 10k, Resistor_SMD:R_0603_1608Metric_Pad0.98x0.95mm_HandSolder, F.Cu at (165.7, 64.0)
- added R4: 10k, Resistor_SMD:R_0603_1608Metric_Pad0.98x0.95mm_HandSolder, F.Cu at (165.7, 65.6)
- added R5: 10k, Resistor_SMD:R_0603_1608Metric_Pad0.98x0.95mm_HandSolder, F.Cu at (133.1, 56.6)
- added R6: 1k, Resistor_SMD:R_0603_1608Metric_Pad0.98x0.95mm_HandSolder, F.Cu at (133.1, 58.2)
- added R7: 1k, Resistor_SMD:R_0603_1608Metric_Pad0.98x0.95mm_HandSolder, F.Cu at (158.3, 48.7)
- added R8: 1k, Resistor_SMD:R_0603_1608Metric_Pad0.98x0.95mm_HandSolder, F.Cu at (136.5, 48.8)
- added R9: 49.9, Resistor_SMD:R_0603_1608Metric_Pad0.98x0.95mm_HandSolder, F.Cu at (147.5, 69.6)
- added SW1: nRST_SW, Button_Switch_THT:SW_PUSH_6mm, F.Cu at (129.8, 67.5)
- added U1: LAN8720A, Package_DFN_QFN:VQFN-24-1EP_4x4mm_P0.5mm_EP2.5x2.5mm_ThermalVias, F.Cu at (147.0, 80.4)
- added Y1: 25MHz, 0_oscillators:01.X.SD.120MMOI025000000, F.Cu at (135.8, 74.0)
Routing:
- net /Project Architecture/LAN8742A breakout/LED2: track 0.00 -> 50.3 mm
- net /Project Architecture/LAN8742A breakout/nRST: track 0.00 -> 44.4 mm, vias 0 -> 2
- net /Project Architecture/LAN8742A breakout/LED1: track 0.00 -> 35.6 mm
- net Net-(JP1-A): track 0.00 -> 33.8 mm, vias 0 -> 2
- net Net-(JP2-B): track 0.00 -> 27.6 mm, vias 0 -> 2
- net +3V3_PHYA: track 0.00 -> 24.6 mm, vias 0 -> 2
- net /Project Architecture/LAN8742A breakout/RX_P: track 0.00 -> 22.5 mm
- net /Project Architecture/LAN8742A breakout/TX_P: track 0.00 -> 22.4 mm
- net /Project Architecture/LAN8742A breakout/TX_N: track 0.00 -> 20.8 mm, vias 0 -> 1
- net /Project Architecture/LAN8742A breakout/RX_N: track 0.00 -> 20.8 mm, vias 0 -> 1
- net /Project Architecture/LAN8742A breakout/TXD1: track 0.00 -> 14.6 mm
- net /Project Architecture/LAN8742A breakout/RXD1: track 0.00 -> 14.2 mm
- net Net-(U1-XTAL1/CLKIN): track 0.00 -> 14.2 mm
- net /Project Architecture/LAN8742A breakout/TXD0: track 0.00 -> 13.3 mm
- net /Project Architecture/LAN8742A breakout/RXD0: track 0.00 -> 12.9 mm
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- added copper zone on B.Cu, net GND
- added copper zone on F.Cu, net GND
- added copper zone on In1.Cu, net GND
- added copper zone on In2.Cu, net GND
Other:
- board outline added: 40 x 50 mm
- copper layers 6 -> 4
- board text removed: "30°"
